File: interface.kicad_sch (KiCad schematic)
At the start: 50 parts

Commit message: Fixes suggested in review
Parts:
- removed U?: TCA9548ARGER, antmicro-footprints:VQFN-24, symbol antmicroLogicSignalSwitchesMultiplexersDecoders:TCA9548ARGER
- added C? (x2): C_100n_0402, antmicro-footprints:0402-cap, symbol antmicroCapacitors0402:C_100n_0402
- added R? (x2): R_2k_0402, antmicro-footprints:0402-res, symbol antmicroResistors0402:R_2k_0402
- added R? (x2): R_0R_0402, antmicro-footprints:0402-res, symbol antmicroResistors0402:R_0R_0402
- added R?: R_10k_0402, antmicro-footprints:0402-res, symbol antmicroResistors0402:R_10k_0402
- added U?: NTS0102DP, antmicro-footprints:TSSOP-8_W3mm, symbol antmicroLogicTranslatorsLevelShifters:NTS0102DP
- added U?: PCA9547BS,118, antmicro-footprints:HVQFN24, symbol antmicroLogicSignalSwitchesMultiplexersDecoders:PCA9547BS,118
Connections:
- net +1V8: now also C?.1, U?.3 (VCC_A), U?.6 (OE); no longer C?.1
- net +3V3: now also C?.1, C?.1, R?.2, R?.2, R?.2, R?.2, U?.21 (VCC), U?.7 (VCC_B)
- net BRIDGE_I2C_SCL: now also U?.15 (SC6)
- net BRIDGE_I2C_SDA: now also U?.14 (SD6)
- net CAM3_SCL: no longer R?.1, R?.1, R?.1, R?.2, R?.2, R?.2, TP?.1, TP?.1, TP?.1
- net CAM3_SDA: no longer R?.1, R?.1, R?.1, R?.2, R?.2, R?.2, TP?.1, TP?.1, TP?.1
- net GND: now also C?.2, C?.2, R?.1, U?.18 (A2), U?.2 (GND), U?.23 (A1), U?.25 (GND), U?.9 (GND)
- net I2C_GP3_CLK: now also U?.4 (A2); no longer R?.1
- net I2C_GP3_DAT: now also U?.5 (A1); no longer R?.1
- net MISC_I2C_SCL: now also U?.17 (SC7)
- net MISC_I2C_SDA: now also U?.16 (SD7)
- net at R?.2: now also U?.20 (SDA)
- net at R?.1: now also U?.4 (SC1)
- net at R?.1: now also U?.5 (SD2)
- net at R?.1: now also U?.8 (SC3)
- net at R?.1: now also U?.1 (SD0)
- net at R?.2: now also U?.19 (SCL)
- net at R?.1: now also U?.2 (SC0)
- net at R?.1: now also U?.3 (SD1)
- net at R?.1: now also U?.6 (SC2)
- net at R?.1: now also U?.7 (SD3)
- new net: R?.1, R?.2, U?.22 (A0)
- new net: R?.1, U?.24 (~{RESET})
- new net CAM0_SCL: R?.1, R?.2, TP?.1
- new net CAM0_SDA: R?.1, R?.2, TP?.1
- new net CAM1_SCL: R?.1, R?.2, TP?.1
- new net CAM1_SDA: R?.1, R?.2, TP?.1
- new net CAM2_SCL: R?.1, R?.2, TP?.1
- new net CAM2_SDA: R?.1, R?.2, TP?.1
- new net SCL_3V3: R?.1, R?.1, U?.1 (B2)
- new net SDA_3V3: R?.1, R?.1, U?.8 (B1)
Other:
- note added: "AGX SoM Camera Connector"
- note added: "I2C Level Shifting"
- note removed: "Motherboard Mezzanine Connector"
- moved on the sheet: C?, TP?
